File: Hardware/THAT-breakouts.brd (EAGLE design)
At the start: 101.6 x 22.9 mm, 27 parts, among them IC1 THAT1206, IC2 THAT1646, J1 INPUT, J2 OUTPUT, J3 CHASSIS

Commit message: More WIP & conceptual work.
Parts:
- added C10, C9: 0.1uF, SparkFun-Capacitors:0603-CAP
- added C11, C12: 10uf, that-ics:PANASONIC_D
- added C7, C8: 100pF, SparkFun-Capacitors:0603-CAP
- added D1, D2: (no value), SparkFun-DiscreteSemi:SOT23-3
- added J5: (no value), SparkFun-Connectors:1X04_NO_SILK_ALL_ROUND
- added JP2: JUMPER-PAD-2-NC_BY_TRACE, SparkFun-Passives:PAD-JUMPER-2-NC_BY_TRACE_YES_SILK
- added L1, L2: 27uH, SparkFun-Passives:0603
- moved FRAME1 131.2 mm to (16.5, -20.3)
- moved IC2 40.5 mm to (61.0, 11.4), turned to 180 degrees
- moved J2 3.59 mm to (101.6, 8.89)
Connections:
- new net N$10: C11.-, D2.3, IC2.8, L2.1
- new net N$11: C12.-, D1.3, IC2.1, L1.1
- new net N$13: C12.+, IC2.2
- new net N$14: C11.+, IC2.7
- new net N$16: IC2.4, J5.4
- new net N$8: C8.1, J2.TIP, L2.2
- new net N$9: C7.1, J2.RING, L1.2
- net GND: now also C10.1, C9.1, J5.1, JP2.2
- net GND-ISO: now also C7.2, C8.2, J2.SLEEVE, JP2.1
- net VCC: now also C9.2, D1.2, D2.2, J5.3
- net VNEG: now also C10.2, D1.1, D2.1, J5.2
Other:
- board size 101.6 x 22.9 mm -> 101.6 x 20.3 mm
- board text added: "IN"

Commit message: Still more WIP.
Parts:
- added J6: CHASSIS, SparkFun-Connectors:1X02_NO_SILK
- moved C7 10.2 mm to (76.2, 6.35), turned to 270 degrees
- moved C8 5.24 mm to (76.2, 14.0), turned to 90 degrees
- moved IC2 1.80 mm to (59.7, 12.7)
- moved L1 1.80 mm to (71.1, 11.4)
- moved D1 1.27 mm to (64.8, 11.4)
- moved C10 1.27 mm to (58.4, 3.81)
- moved C9 1.27 mm to (61.0, 3.81)
- moved D2 1.27 mm to (67.3, 8.89)
- moved J2 1.27 mm to (100.3, 8.89)
- moved L2 1.27 mm to (71.1, 8.89)
- flipped JP1 to the bottom, turned to 180 degrees
Connections:
- net GND-ISO: now also J6.1, J6.2
Other:
- board size 101.6 x 20.3 mm -> 100.3 x 20.3 mm

Commit message: Found some zeners...
Parts:
- added D3, D4: 12V, that-ics:SOD-323
- JP1: value JUMPER-PAD-2-NC_BY_TRACE -> GND-JOIN
- moved D5 3.05 mm to (27.9, 13.5)
- moved C1 2.03 mm to (27.9, 10.7)
- moved R2 2.03 mm to (24.1, 10.7)
- moved D6 1.00 mm to (27.9, 6.08)
- moved C6 0.51 mm to (34.3, 16.0)
Connections:
- new net N$12: D3.A, D5.1, D6.1
- new net N$15: D4.C, D5.2, D6.2
- net VCC: now also D4.A
- net VNEG: now also D3.C
Changed lines of the file:
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@@
 <setting verticaltext="up"/>
 </settings>
-<grid distance="0.05" unitdist="inch" unit="inch" style="lines" multiple="1" display="yes" altdistance="0.005" altunitdist="inch" altunit="inch"/>
+<grid distance="0.01" unitdist="inch" unit="inch" style="lines" multiple="1" display="yes" altdistance="0.005" altunitdist="inch" altunit="inch"/>
 <layers>
 <layer number="1" name="Top" color="4" fill="1" visible="yes" active="yes"/>
@@
 <attribute name="PROD_ID" value="RES-07863" x="24.13" y="8.89" size="1.778" layer="27" font="vector" ratio="15" display="off"/>
 </element>
-<element name="R2" library="SparkFun-Resistors" package="0603-RES" value="100" x="24.13" y="12.7">
-<attribute name="PROD_ID" value="RES-07863" x="24.13" y="12.7" size="1.778" layer="27" font="vector" ratio="15" display="off"/>
+<element name="R2" library="SparkFun-Resistors" package="0603-RES" value="100" x="24.13" y="10.668">
+<attribute name="PROD_ID" value="RES-07863" x="24.13" y="10.668" size="1.778" layer="27" font="vector" ratio="15" display="off"/>
 </element>
 <element name="R3" library="SparkFun-Resistors" package="0603-RES" value="4.7K" x="36.83" y="2.54">
 <attribute name="PROD_ID" value="RES-07857" x="36.83" y="2.54" size="1.778" layer="27" font="vector" ratio="15" display="off"/>
 </element>
-<element name="C1" library="SparkFun-Capacitors" package="0603-CAP" value="470pF" x="27.94" y="12.7">
-<attribute name="PROD_ID" value="CAP-07884" x="27.94" y="12.7" size="1.778" layer="27" font="vector" ratio="15" display="off"/>
+<element name="C1" library="SparkFun-Capacitors" package="0603-CAP" value="470pF" x="27.94" y="10.668">
+<attribute name="PROD_ID" value="CAP-07884" x="27.94" y="10.668" size="1.778" layer="27" font="vector" ratio="15" display="off"/>
 </element>
 <element name="C2" library="SparkFun-Capacitors" package="0603-CAP" value="470pF" x="27.94" y="8.89" rot="R180">
@@
 <attribute name="PROD_ID" value="CAP-07883" x="24.13" y="5.08" size="1.778" layer="27" font="vector" ratio="15" rot="R180" display="off"/>
 </element>
-<element name="JP1" library="SparkFun-Passives" package="PAD-JUMPER-2-NC_BY_TRACE_YES_SILK" value="JUMPER-PAD-2-NC_BY_TRACE" x="24.765" y="2.54" rot="MR180"/>
+<element name="JP1" library="SparkFun-Passives" package="PAD-JUMPER-2-NC_BY_TRACE_YES_SILK" value="GND-JOIN" x="24.765" y="2.54" rot="MR180"/>
 <element name="C4" library="SparkFun-Capacitors" package="0603-CAP" value="0.1uF" x="34.29" y="11.43" rot="R180">
 <attribute name="PROD_ID" value="CAP-08604" x="34.29" y="11.43" size="1.778" layer="27" font="vector" ratio="15" rot="R180" display="off"/>
@@
 <element name="H7" library="SparkFun-Electromechanical" package="STAND-OFF" value="STAND-OFF" x="-119.38" y="-64.77"/>
 <element name="H8" library="SparkFun-Electromechanical" package="STAND-OFF" value="STAND-OFF" x="-119.38" y="-71.12"/>
-<element name="D5" library="SparkFun-DiscreteSemi" package="SOT23-3" value="" x="27.94" y="16.51" rot="R180">
-<attribute name="PROD_ID" value="DIO-10647" x="27.94" y="16.51" size="1.778" layer="27" font="vector" ratio="15" rot="R180" display="off"/>
-</element>
-<element name="D6" library="SparkFun-DiscreteSemi" package="SOT23-3" value="" x="27.94" y="5.08">
-<attribute name="PROD_ID" value="DIO-10647" x="27.94" y="5.08" size="1.778" layer="27" font="vector" ratio="15" display="off"/>
-</element>
-<element name="C6" library="that-ics" package="PANASONIC_D" value="220uf" x="34.29" y="16.51"/>
+<element name="D5" library="SparkFun-DiscreteSemi" package="SOT23-3" value="" x="27.94" y="13.462" rot="R180">
+<attribute name="PROD_ID" value="DIO-10647" x="27.94" y="13.462" size="1.778" layer="27" font="vector" ratio="15" rot="R180" display="off"/>
+</element>
+<element name="D6" library="SparkFun-DiscreteSemi" package="SOT23-3" value="" x="27.94" y="6.08">
+<attribute name="PROD_ID" value="DIO-10647" x="27.94" y="6.08" size="1.778" layer="27" font="vector" ratio="15" display="off"/>
+</element>
+<element name="C6" library="that-ics" package="PANASONIC_D" value="220uf" x="34.29" y="16.002"/>
 <element name="L1" library="SparkFun-Passives" package="0603" value="27uH" x="71.12" y="11.43"/>
 <element name="L2" library="SparkFun-Passives" package="0603" value="27uH" x="71.12" y="8.89"/>
@@
 </element>
 <element name="J6" library="SparkFun-Connectors" package="1X02_NO_SILK" value="CHASSIS" x="97.79" y="7.62" rot="R90"/>
+<element name="D3" library="that-ics" package="SOD-323" value="12V" x="27.94" y="2.54" rot="R180">
+<attribute name="DK_PN" value="MM3Z12VT1GOSCT-ND" x="27.94" y="2.54" size="1.778" layer="27" font="vector" ratio="15" rot="R180" display="off"/>
+<attribute name="MFR_PN" value="MM3Z12VT1G" x="27.94" y="2.54" size="1.778" layer="27" font="vector" ratio="15" rot="R180" display="off"/>
+<attribute name="MFR" value="ON Semi" x="27.94" y="2.54" size="1.778" layer="27" font="vector" ratio="15" rot="R180" display="off"/>
+</element>
+<element name="D4" library="that-ics" package="SOD-323" value="12V" x="27.94" y="17.018">
+<attribute name="DK_PN" value="MM3Z12VT1GOSCT-ND" x="27.94" y="17.018" size="1.778" layer="27" font="vector" ratio="15" display="off"/>
+<attribute name="MFR_PN" value="MM3Z12VT1G" x="27.94" y="17.018" size="1.778" layer="27" font="vector" ratio="15" display="off"/>
+<attribute name="MFR" value="ON Semi" x="27.94" y="17.018" size="1.778" layer="27" font="vector" ratio="15" display="off"/>
+</element>
 </elements>
 <signals>
@@
 <contactref element="C10" pad="2"/>
 <contactref element="J5" pad="2"/>
+<contactref element="D3" pad="C"/>
 <wire x1="66.36" y1="7.89" x2="65.72" y2="12.43" width="0" layer="19" extent="1-1"/>
 <wire x1="57.785" y1="10.0838" x2="65.72" y2="12.43" width="0" layer="19" extent="1-1"/>
@@
 <wire x1="31.6738" y1="5.715" x2="44.45" y2="8.89" width="0" layer="19" extent="1-1"/>
 <wire x1="30.9" y1="2.54" x2="31.6738" y2="5.715" width="0" layer="19" extent="1-1"/>
+<wire x1="29.09" y1="2.54" x2="30.9" y2="2.54" width="0" layer="19" extent="1-1"/>
 </signal>
 <signal name="GND">
@@
 <contactref element="C9" pad="2"/>
 <contactref element="J5" pad="3"/>
+<contactref element="D4" pad="A"/>
 <wire x1="59.055" y1="10.0838" x2="63.82" y2="12.43" width="0" layer="19" extent="1-1"/>
 <wire x1="60.96" y1="4.66" x2="59.055" y2="10.0838" width="0" layer="19" extent="1-1"/>
@@
 <wire x1="36.9062" y1="8.255" x2="44.45" y2="11.43" width="0" layer="19" extent="1-1"/>
 <wire x1="35.14" y1="11.43" x2="36.9062" y2="8.255" width="0" layer="19" extent="1-1"/>
+<wire x1="29.09" y1="17.018" x2="35.14" y2="11.43" width="0" layer="19" extent="1-1"/>
 </signal>
 <signal name="N$1">
 <contactref element="J1" pad="RING"/>
 <contactref element="R2" pad="1"/>
-<wire x1="10.5" y1="4.48" x2="23.28" y2="12.7" width="0" layer="19" extent="1-1"/>
+<wire x1="10.5" y1="4.48" x2="23.28" y2="10.668" width="0" layer="19" extent="1-1"/>
 </signal>
 <signal name="N$2">
@@
 <contactref element="C1" pad="1"/>
 <contactref element="D5" pad="3"/>
-<wire x1="27.09" y1="12.7" x2="27.94" y2="15.41" width="0" layer="19" extent="1-1"/>
-<wire x1="24.98" y1="12.7" x2="27.09" y2="12.7" width="0" layer="19" extent="1-1"/>
-<wire x1="31.6738" y1="8.255" x2="27.09" y2="12.7" width="0" layer="19" extent="1-1"/>
+<wire x1="27.09" y1="10.668" x2="31.6738" y2="8.255" width="0" layer="19" extent="1-1"/>
+<wire x1="27.94" y1="12.362" x2="27.09" y2="10.668" width="0" layer="19" extent="1-1"/>
+<wire x1="24.98" y1="10.668" x2="27.09" y2="10.668" width="0" layer="19" extent="1-1"/>
 </signal>
 <signal name="N$3">
@@
 <contactref element="C2" pad="2"/>
 <contactref element="D6" pad="3"/>
-<wire x1="27.94" y1="6.18" x2="31.6738" y2="6.985" width="0" layer="19" extent="1-1"/>
-<wire x1="27.09" y1="8.89" x2="27.94" y2="6.18" width="0" layer="19" extent="1-1"/>
+<wire x1="27.94" y1="7.18" x2="31.6738" y2="6.985" width="0" layer="19" extent="1-1"/>
+<wire x1="27.09" y1="8.89" x2="27.94" y2="7.18" width="0" layer="19" extent="1-1"/>
 <wire x1="24.98" y1="8.89" x2="27.09" y2="8.89" width="0" layer="19" extent="1-1"/>
 </signal>
@@
 <contactref element="R3" pad="1"/>
 <contactref element="C3" pad="1"/>
-<wire x1="28.79" y1="8.89" x2="28.79" y2="12.7" width="0" layer="19" extent="1-1"/>
+<wire x1="28.79" y1="8.89" x2="28.79" y2="10.668" width="0" layer="19" extent="1-1"/>
 <wire x1="24.98" y1="5.08" x2="28.79" y2="8.89" width="0" layer="19" extent="1-1"/>
 <wire x1="35.98" y1="2.54" x2="28.79" y2="8.89" width="0" layer="19" extent="1-1"/>
@@
 <contactref element="IC1" pad="5"/>
 <contactref element="C6" pad="-"/>
-<wire x1="36.9062" y1="5.715" x2="31.89" y2="16.51" width="0" layer="19" extent="1-1"/>
+<wire x1="36.9062" y1="5.715" x2="31.89" y2="16.002" width="0" layer="19" extent="1-1"/>
 <wire x1="37.68" y1="2.54" x2="36.9062" y2="5.715" width="0" layer="19" extent="1-1"/>
 </signal>
@@
 <contactref element="IC1" pad="8"/>
 <contactref element="C6" pad="+"/>
-<wire x1="36.9062" y1="9.525" x2="36.69" y2="16.51" width="0" layer="19" extent="1-1"/>
+<wire x1="36.9062" y1="9.525" x2="36.69" y2="16.002" width="0" layer="19" extent="1-1"/>
 </signal>
 <signal name="N$8">
@@
 <wire x1="53.34" y1="13.97" x2="57.785" y2="15.3162" width="0" layer="19" extent="1-1"/>
 </signal>
+<signal name="N$12">
+<contactref element="D3" pad="A"/>
+<contactref element="D5" pad="1"/>
+<contactref element="D6" pad="1"/>
+<wire x1="26.99" y1="5.08" x2="28.89" y2="14.462" width="0" layer="19" extent="1-1"/>
+<wire x1="26.79" y1="2.54" x2="26.99" y2="5.08" width="0" layer="19" extent="1-1"/>
+</signal>
+<signal name="N$15">
+<contactref element="D6" pad="2"/>
+<contactref element="D5" pad="2"/>
+<contactref element="D4" pad="C"/>
+<wire x1="26.99" y1="14.462" x2="26.79" y2="17.018" width="0" layer="19" extent="1-1"/>
+<wire x1="28.89" y1="5.08" x2="26.99" y2="14.462" width="0" layer="19" extent="1-1"/>
+</signal>
 </signals>
