File: Hardware/THAT-breakouts.sch (EAGLE design)
At the start: 27 parts, among them IC1 THAT1206, IC2 THAT1646, J1 INPUT, J2 OUTPUT, J3 CHASSIS

Commit message: More WIP & conceptual work.
Parts:
- added C10, C9: 0.1uF, SparkFun-Capacitors:0.1UF-25V-5%(0603)
- added C11, C12: 10uf, that-ics:PANA-EEE-1EA100NP
- added C7, C8: 100pF, SparkFun-Capacitors:100PF-50V-5%(0603)
- added D1, D2: (no value), SparkFun-DiscreteSemi:BAV99
- added J5: (no value), SparkFun-Connectors:M04NO_SILK_ALL_ROUND
- added JP2: JUMPER-PAD-2-NC_BY_TRACE, SparkFun-Passives:JUMPER-PAD-2-NC_BY_TRACE
- added L1, L2: 27uH, SparkFun-Passives:INDUCTOR0603
Connections:
- new net N$10: C11.-, D2.COM, IC2.OUT+, L2.1
- new net N$11: C12.-, D1.COM, IC2.OUT-, L1.1
- new net N$13: C12.+, IC2.SNS-
- new net N$14: C11.+, IC2.SNS+
- new net N$16: IC2.IN, J5.4
- new net N$8: C8.1, J2.TIP, L2.2
- new net N$9: C7.1, J2.RING, L1.2
- net GND: now also C10.1, C9.1, J5.1, JP2.2
- net GND-ISO: now also C7.2, C8.2, J2.EARTH, JP2.1
- net VCC: now also C9.2, D1.C2, D2.C2, J5.3
- net VNEG: now also C10.2, D1.A1, D2.A1, J5.2
Other:
- moved on the sheet: C1, C2, C3, C4, C5, C6, IC1, IC2, J1, J2, J3, J4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

Commit message: Still more WIP.
Parts:
- added J6: CHASSIS, SparkFun-Connectors:M021X02_NO_SILK
Connections:
- net GND-ISO: now also J6.1, J6.2
Other:
- moved on the sheet: J2
Changed lines of the file:
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@@
 <part name="SUPPLY13" library="SparkFun-Aesthetics" deviceset="VNEG" device=""/>
 <part name="SUPPLY14" library="SparkFun-Aesthetics" deviceset="VCC" device=""/>
+<part name="J6" library="SparkFun-Connectors" deviceset="M02" device="1X02_NO_SILK" value="CHASSIS"/>
 </parts>
 <sheets>
@@
 <instance part="FRAME1" gate="V" x="147.32" y="0"/>
 <instance part="J1" gate="G$1" x="22.86" y="142.24" rot="MR180"/>
-<instance part="J2" gate="G$1" x="203.2" y="66.04" rot="R180"/>
+<instance part="J2" gate="G$1" x="203.2" y="68.58" rot="R180"/>
 <instance part="SUPPLY1" gate="G$1" x="119.38" y="162.56"/>
 <instance part="SUPPLY3" gate="G$1" x="96.52" y="73.66"/>
@@
 <instance part="SUPPLY13" gate="G$2" x="66.04" y="30.48"/>
 <instance part="SUPPLY14" gate="G$1" x="60.96" y="53.34"/>
+<instance part="J6" gate="G$1" x="208.28" y="53.34" rot="R180"/>
 </instances>
 <busses>
@@
 <wire x1="195.58" y1="43.18" x2="195.58" y2="48.26" width="0.1524" layer="91"/>
 <pinref part="J2" gate="G$1" pin="EARTH"/>
-<wire x1="195.58" y1="48.26" x2="195.58" y2="58.42" width="0.1524" layer="91"/>
-<wire x1="195.58" y1="58.42" x2="198.12" y2="58.42" width="0.1524" layer="91"/>
+<wire x1="195.58" y1="48.26" x2="195.58" y2="50.8" width="0.1524" layer="91"/>
+<wire x1="195.58" y1="50.8" x2="195.58" y2="53.34" width="0.1524" layer="91"/>
+<wire x1="195.58" y1="53.34" x2="195.58" y2="60.96" width="0.1524" layer="91"/>
+<wire x1="195.58" y1="60.96" x2="198.12" y2="60.96" width="0.1524" layer="91"/>
 <pinref part="C8" gate="G$1" pin="2"/>
 <wire x1="175.26" y1="50.8" x2="175.26" y2="48.26" width="0.1524" layer="91"/>
@@
 <wire x1="185.42" y1="50.8" x2="185.42" y2="48.26" width="0.1524" layer="91"/>
 <junction x="185.42" y="48.26"/>
+<pinref part="J6" gate="G$1" pin="1"/>
+<wire x1="200.66" y1="53.34" x2="195.58" y2="53.34" width="0.2032" layer="91"/>
+<pinref part="J6" gate="G$1" pin="2"/>
+<wire x1="195.58" y1="50.8" x2="200.66" y2="50.8" width="0.2032" layer="91"/>
+<junction x="195.58" y="50.8"/>
+<junction x="195.58" y="53.34"/>
+<junction x="195.58" y="48.26"/>
 </segment>
 <segment>
@@
 <wire x1="172.72" y1="63.5" x2="175.26" y2="63.5" width="0.1524" layer="91"/>
 <pinref part="C8" gate="G$1" pin="1"/>
-<wire x1="175.26" y1="63.5" x2="198.12" y2="63.5" width="0.1524" layer="91"/>
+<wire x1="175.26" y1="63.5" x2="190.5" y2="63.5" width="0.1524" layer="91"/>
+<wire x1="190.5" y1="63.5" x2="190.5" y2="66.04" width="0.1524" layer="91"/>
+<wire x1="190.5" y1="66.04" x2="198.12" y2="66.04" width="0.1524" layer="91"/>
 <wire x1="175.26" y1="63.5" x2="175.26" y2="58.42" width="0.1524" layer="91"/>
 <junction x="175.26" y="63.5"/>
@@
 <segment>
 <pinref part="J2" gate="G$1" pin="RING"/>
-<wire x1="198.12" y1="68.58" x2="190.5" y2="68.58" width="0.1524" layer="91"/>
-<wire x1="190.5" y1="68.58" x2="190.5" y2="71.12" width="0.1524" layer="91"/>
+<wire x1="198.12" y1="71.12" x2="185.42" y2="71.12" width="0.1524" layer="91"/>
 <pinref part="L1" gate="G$1" pin="2"/>
-<wire x1="190.5" y1="71.12" x2="185.42" y2="71.12" width="0.1524" layer="91"/>
 <pinref part="C7" gate="G$1" pin="1"/>
 <wire x1="185.42" y1="71.12" x2="172.72" y2="71.12" width="0.1524" layer="91"/>

Commit message: Found some zeners...
Parts:
- added D3, D4: 12V, that-ics:12V-ZENER-DIODE
- JP1: value JUMPER-PAD-2-NC_BY_TRACE -> GND-JOIN
Connections:
- new net N$12: D3.A, D5.A1, D6.A1
- new net N$15: D4.C, D5.C2, D6.C2
- net VCC: now also D4.A
- net VNEG: now also D3.C
Other:
- moved on the sheet: JP1
Changed lines of the file:
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@@
 <part name="C2" library="SparkFun-Capacitors" deviceset="470PF-50V-5%(0603)" device="SMD" value="470pF"/>
 <part name="C3" library="SparkFun-Capacitors" deviceset="100PF-50V-5%(0603)" device="" value="100pF"/>
-<part name="JP1" library="SparkFun-Passives" deviceset="JUMPER-PAD-2-NC_BY_TRACE" device=""/>
+<part name="JP1" library="SparkFun-Passives" deviceset="JUMPER-PAD-2-NC_BY_TRACE" device="" value="GND-JOIN"/>
 <part name="GND4" library="SparkFun-Aesthetics" deviceset="GND-ISO" device=""/>
 <part name="GND5" library="SparkFun-Aesthetics" deviceset="GND-ISO" device=""/>
@@
 <part name="SUPPLY14" library="SparkFun-Aesthetics" deviceset="VCC" device=""/>
 <part name="J6" library="SparkFun-Connectors" deviceset="M02" device="1X02_NO_SILK" value="CHASSIS"/>
+<part name="D3" library="that-ics" deviceset="12V-ZENER-DIODE" device="" value="12V"/>
+<part name="D4" library="that-ics" deviceset="12V-ZENER-DIODE" device="" value="12V"/>
 </parts>
 <sheets>
@@
 <instance part="C2" gate="G$1" x="60.96" y="124.46"/>
 <instance part="C3" gate="G$1" x="68.58" y="111.76"/>
-<instance part="JP1" gate="G$1" x="160.02" y="101.6" rot="MR0"/>
+<instance part="JP1" gate="G$1" x="93.98" y="109.22"/>
 <instance part="GND4" gate="G$1" x="68.58" y="104.14"/>
-<instance part="GND5" gate="G$1" x="167.64" y="96.52" rot="MR0"/>
-<instance part="GND6" gate="1" x="152.4" y="96.52" rot="MR0"/>
+<instance part="GND5" gate="G$1" x="86.36" y="99.06"/>
+<instance part="GND6" gate="1" x="104.14" y="99.06"/>
 <instance part="C4" gate="G$1" x="129.54" y="160.02" rot="R90"/>
 <instance part="C5" gate="G$1" x="129.54" y="116.84" rot="R90"/>
@@
 <instance part="GND9" gate="1" x="114.3" y="114.3"/>
 <instance part="J3" gate="G$1" x="17.78" y="121.92"/>
-<instance part="SUPPLY2" gate="G$1" x="116.84" y="177.8"/>
-<instance part="SUPPLY4" gate="G$2" x="68.58" y="154.94"/>
+<instance part="SUPPLY2" gate="G$1" x="137.16" y="177.8"/>
+<instance part="SUPPLY4" gate="G$2" x="50.8" y="160.02"/>
 <instance part="J4" gate="G$1" x="160.02" y="124.46" rot="MR0"/>
 <instance part="GND10" gate="1" x="152.4" y="114.3"/>
@@
 <instance part="SUPPLY14" gate="G$1" x="60.96" y="53.34"/>
 <instance part="J6" gate="G$1" x="208.28" y="53.34" rot="R180"/>
+<instance part="D3" gate="G$1" x="58.42" y="165.1" rot="R180"/>
+<instance part="D4" gate="G$1" x="129.54" y="175.26" rot="R180"/>
 </instances>
 <busses>
@@
 <pinref part="SUPPLY13" gate="G$2" pin="VNEG"/>
 </segment>
+<segment>
+<pinref part="SUPPLY4" gate="G$2" pin="VNEG"/>
+<pinref part="D3" gate="G$1" pin="C"/>
+<wire x1="50.8" y1="162.56" x2="50.8" y2="165.1" width="0.1524" layer="91"/>
+<wire x1="50.8" y1="165.1" x2="55.88" y2="165.1" width="0.1524" layer="91"/>
+</segment>
 </net>
 <net name="GND" class="0">
@@
 <segment>
 <pinref part="GND6" gate="1" pin="GND"/>
-<wire x1="152.4" y1="99.06" x2="152.4" y2="101.6" width="0.1524" layer="91"/>
+<wire x1="104.14" y1="101.6" x2="104.14" y2="109.22" width="0.1524" layer="91"/>
 <pinref part="JP1" gate="G$1" pin="2"/>
-<wire x1="152.4" y1="101.6" x2="154.94" y2="101.6" width="0.1524" layer="91"/>
+<wire x1="104.14" y1="109.22" x2="99.06" y2="109.22" width="0.1524" layer="91"/>
 </segment>
 <segment>
@@
 <pinref part="SUPPLY14" gate="G$1" pin="VCC"/>
 <wire x1="60.96" y1="45.72" x2="60.96" y2="53.34" width="0.1524" layer="91"/>
+</segment>
+<segment>
+<pinref part="D4" gate="G$1" pin="A"/>
+<pinref part="SUPPLY2" gate="G$1" pin="VCC"/>
+<wire x1="132.08" y1="175.26" x2="137.16" y2="175.26" width="0.1524" layer="91"/>
+<wire x1="137.16" y1="175.26" x2="137.16" y2="177.8" width="0.1524" layer="91"/>
 </segment>
 </net>
@@
 <segment>
 <pinref part="GND5" gate="G$1" pin="GND-ISO"/>
-<wire x1="167.64" y1="99.06" x2="167.64" y2="101.6" width="0.1524" layer="91"/>
+<wire x1="86.36" y1="101.6" x2="86.36" y2="109.22" width="0.1524" layer="91"/>
 <pinref part="JP1" gate="G$1" pin="1"/>
-<wire x1="167.64" y1="101.6" x2="165.1" y2="101.6" width="0.1524" layer="91"/>
+<wire x1="86.36" y1="109.22" x2="88.9" y2="109.22" width="0.1524" layer="91"/>
 </segment>
 <segment>
@@
 </segment>
 </net>
+<net name="N$12" class="0">
+<segment>
+<pinref part="D3" gate="G$1" pin="A"/>
+<wire x1="60.96" y1="165.1" x2="63.5" y2="165.1" width="0.1524" layer="91"/>
+<pinref part="D5" gate="G$1" pin="A1"/>
+<wire x1="63.5" y1="165.1" x2="63.5" y2="175.26" width="0.1524" layer="91"/>
+<wire x1="63.5" y1="175.26" x2="93.98" y2="175.26" width="0.1524" layer="91"/>
+<pinref part="D6" gate="G$1" pin="A1"/>
+<wire x1="76.2" y1="165.1" x2="63.5" y2="165.1" width="0.1524" layer="91"/>
+<junction x="63.5" y="165.1"/>
+</segment>
+</net>
+<net name="N$15" class="0">
+<segment>
+<pinref part="D6" gate="G$1" pin="C2"/>
+<wire x1="96.52" y1="165.1" x2="116.84" y2="165.1" width="0.1524" layer="91"/>
+<wire x1="116.84" y1="165.1" x2="116.84" y2="175.26" width="0.1524" layer="91"/>
+<pinref part="D5" gate="G$1" pin="C2"/>
+<wire x1="116.84" y1="175.26" x2="114.3" y2="175.26" width="0.1524" layer="91"/>
+<pinref part="D4" gate="G$1" pin="C"/>
+<wire x1="116.84" y1="175.26" x2="127" y2="175.26" width="0.1524" layer="91"/>
+<junction x="116.84" y="175.26"/>
+</segment>
+</net>
