File: Hardware/THAT_1646_Breakout.sch (EAGLE design)
At the start: 42 parts, among them IC1 THAT1206, IC2 THAT1646, J1 INPUT, J2 OUTPUT, J3 CHASSIS, J6 CHASSIS

Commit message: Broke into 2 separate board files.
Parts:
- removed C1, C2: 470pF, SparkFun-Capacitors:470PF-50V-5%(0603)SMD
- removed C3: 100pF, SparkFun-Capacitors:100PF-50V-5%(0603)
- removed C4, C5: 0.1uF, SparkFun-Capacitors:0.1UF-25V-5%(0603)
- removed C6: 220uf, that-ics:PANA-EEE-FKOJ221P
- removed D3, D4: 12V, that-ics:12V-ZENER-DIODE
- removed D5, D6: (no value), SparkFun-DiscreteSemi:BAV99
- removed H1, H2, H3, H4: STAND-OFF, SparkFun-Electromechanical:STAND-OFF
- removed IC1: THAT1206, that-ics:THAT1206
- removed J1: INPUT, SparkFun-Connectors:AUDIO-JACK4-.25-HORIZ-TRS
- removed J3: CHASSIS, SparkFun-Connectors:M021X02_NO_SILK
- removed J4: (no value), SparkFun-Connectors:M04NO_SILK_ALL_ROUND
- removed JP1: GND-JOIN, SparkFun-Passives:JUMPER-PAD-2-NC_BY_TRACE
- removed R1, R2: 100, SparkFun-Resistors:100OHM-1/10W-1%(0603)
- removed R3: 4.7K, SparkFun-Resistors:4.7KOHM-1/10W-1%(0603)
Connections:
- removed net N$1: J1.RING, R2.1
- removed net N$12: D3.A, D5.A1, D6.A1
- removed net N$15: D4.C, D5.C2, D6.C2
- removed net N$2: C1.1, D5.COM, IC1.IN-, R2.2
- removed net N$3: J1.TIP, R1.1
- removed net N$4: C2.2, D6.COM, IC1.IN+, R1.2
- removed net N$5: C1.2, C2.1, C3.1, R3.1
- removed net N$6: C6.-, IC1.CMIN, R3.2
- removed net N$7: C6.+, IC1.CMOUT
- removed net RCV: IC1.OUT, J4.4
- net GND: no longer C4.2, C5.2, IC1.REF, J4.1, JP1.2
- net GND-ISO: no longer C3.2, J1.EARTH, J3.1, J3.2, JP1.1
- net VCC: no longer C4.1, D4.A, IC1.VCC, J4.3
- net VNEG: no longer C5.1, D3.C, IC1.VEE, J4.2
Other:
- note added: "Chassis ground region"
- note added: "Circuit ground region"
- note added: "How to use JP1, a note on grounding & shielding: For prototyping/breadboarding, the entire board is grounded through the output connector (J4). In that case, leave JP1 intact. If installing in a metal enclosure, the enclosure should be tied to earth, and the shield should be toed to the enclosure as directly as possible. In this case, cut JP1, and run a heavy wire from J3 to the chassis. This avo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"
- note added: "This board requires bipolar power, in the range from +/-5VDC to +/-20VDC."
- note added: "V01"
- moved on the sheet: C10, C11, C12, C7, C8, C9, D1, D2, IC2, J2, J5, J6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
